Commit message: Revert "add some changes to rendering"
This reverts commit eb638a5785cb59885c3a5856f4478c47dab82388.

File: mocca_envs/data/objects/misc/left_foot.urdf (robot description, URDF)
Before this commit: robot foot, 1 links, 0 joints
Links:
- link base_link: geometry visual box size=1 0.5 0.02; visual box size=1.5 1 0.02

Commit message: update step rendering

File: mocca_envs/data/objects/misc/left_foot.urdf (robot description, URDF)
Before this commit: robot foot, 1 links, 0 joints
Links:
- link base_link: geometry visual mesh filename=triangle.stl scale=2 2 2
